File: framos_FSM_IMX_2LANE_Jetson_Adapter.sch (KiCad schematic (older format))
At the start: 27 parts, among them J1 DF40HC(4.0)-60DS-0.4V(51), J2 1-1734248-5, P1 53261-0371, U1 MIC5259-1.8YD5-TR, U2 LP5907MFX-1.2, U3 PCA9306D_118, X1 TXC-7C

Commit message: Add documentation
Connections:
- wire segments 177 -> 181
Changed lines of the file:
@@
 	7020 4065 7020 4545
-Wire Wire Line
-	7020 3730 7020 4065
 Wire Wire Line
 	10170 4040 10170 4645
@@
 	1    0    0    -1
 $EndComp
+Wire Wire Line
+	7020 3780 9900 3780
+Wire Wire Line
+	9900 3780 9900 3000
+Wire Wire Line
+	9900 3000 9990 3000
+Wire Wire Line
+	7020 3730 7020 3780
+Wire Wire Line
+	7020 3780 7020 4065
+Connection ~ 7020 3780
 $EndSCHEMATC
